File: pcb/rc-controller.kicad_sch (KiCad schematic)
At the start: 79 parts, among them J2 USB_C_Receptacle_USB2.0_16P, M1 Motor_DC, Q1 AO3401A, Q2 AO3401A, Q3 AO3400A, Q4 AO3400A, SW1 SW_SPDT, SW2 SW_SPDT, SW3 SW_Push, SW4 SW_Push, SW5 SW_Push, SW6 SW_Push, U1 STM32F401RCTx, U2 LPS22HB, U3 SRV05-4, U4 TX4401, U5 ICM-42670-P, U6 TP4057-42, U7 nrf24L01P_PA_LNA, U8 SSD1306, Y1 16MHz

Commit message: Add net classes
Connections:
- net TSW1A: no longer SW1.1 (A)
- net TSW1B: no longer SW1.3 (C)
- net TSW2A: no longer SW2.1 (A)
- net TSW2B: no longer SW2.3 (C)
- net BT1 renamed BTN1
- net BT2 renamed BTN2
- net BT3 renamed BTN3
- net BT4 renamed BTN4
- net OSCIN renamed XTALH
- net OSCLO renamed XTALC
- net OSCOUT renamed XTALL
- net PWRON renamed BON
- new net SW1A: SW1.1 (A)
- new net SW1B: SW1.3 (C)
- new net SW2A: SW2.1 (A)
- new net SW2B: SW2.3 (C)
Changed lines of the file:
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@@
 	)
 	(junction
-		(at 129.54 265.43)
-		(diameter 0)
-		(color 0 0 0 0)
-	)
-	(junction
 		(at 52.07 180.34)
 		(diameter 0)
@@
 	(wire
 		(pts
-			(xy 129.54 265.43) (xy 127 265.43)
-		)
-		(stroke
-			(width 0)
-			(type default)
-		)
-	)
-	(wire
-		(pts
 			(xy 82.55 88.9) (xy 69.85 88.9)
 		)
@@
 	(wire
 		(pts
-			(xy 127 265.43) (xy 127 262.89)
-		)
-		(stroke
-			(width 0)
-			(type default)
-		)
-	)
-	(wire
-		(pts
 			(xy 175.26 77.47) (xy 180.34 77.47)
 		)
@@
 	(wire
 		(pts
-			(xy 129.54 265.43) (xy 129.54 267.97)
-		)
-		(stroke
-			(width 0)
-			(type default)
-		)
-	)
-	(wire
-		(pts
 			(xy 144.78 247.65) (xy 152.4 247.65)
 		)
@@
 		)
 	)
-	(label "OSCOUT"
+	(label "XTALL"
 		(at 347.98 165.1 0)
 		(fields_autoplaced yes)
@@
 		)
 	)
+	(label "SW2B"
+		(at 218.44 43.18 0)
+		(fields_autoplaced yes)
+		(effects
+			(font
+				(size 1.27 1.27)
+			)
+			(justify left bottom)
+		)
+	)
 	(label "SDA"
 		(at 240.03 203.2 0)
@@
 		)
 	)
-	(label "TSW2A"
-		(at 217.17 38.1 0)
+	(label "SW2A"
+		(at 218.44 38.1 0)
 		(fields_autoplaced yes)
 		(effects
@@
 		)
 	)
-	(label "BT3"
+	(label "BTN3"
 		(at 175.26 77.47 0)
 		(fields_autoplaced yes)
@@
 		)
 	)
-	(label "BT4"
+	(label "BTN4"
 		(at 330.2 87.63 0)
 		(fields_autoplaced yes)
@@
 		)
 	)
-	(label "OSCIN"
+	(label "XTALH"
 		(at 316.23 189.23 0)
 		(fields_autoplaced yes)
@@
 		)
 	)
-	(label "BT2"
+	(label "BTN2"
 		(at 200.66 58.42 0)
 		(fields_autoplaced yes)
@@
 		)
 	)
-	(label "TSW1A"
-		(at 191.77 38.1 0)
-		(fields_autoplaced yes)
-		(effects
-			(font
-				(size 1.27 1.27)
-			)
-			(justify left bottom)
-		)
-	)
 	(label "RE1B"
 		(at 171.45 124.46 0)
@@
 		)
 	)
+	(label "SW1B"
+		(at 193.04 43.18 0)
+		(fields_autoplaced yes)
+		(effects
+			(font
+				(size 1.27 1.27)
+			)
+			(justify left bottom)
+		)
+	)
 	(label "JY1SW"
 		(at 266.7 35.56 0)
@@
 		)
 	)
-	(label "BT3"
+	(label "BTN3"
 		(at 330.2 85.09 0)
 		(fields_autoplaced yes)
@@
 		)
 	)
-	(label "PWRON"
-		(at 309.88 74.93 0)
+	(label "SNMOSI"
+		(at 194.31 259.08 0)
 		(fields_autoplaced yes)
 		(effects
@@
 		)
 	)
-	(label "SNMOSI"
-		(at 194.31 259.08 0)
+	(label "MTR"
+		(at 162.56 170.18 0)
 		(fields_autoplaced yes)
 		(effects
@@
 		)
 	)
-	(label "MTR"
-		(at 162.56 170.18 0)
+	(label "SNSBUS"
+		(at 102.87 87.63 0)
 		(fields_autoplaced yes)
 		(effects
@@
 		)
 	)
-	(label "SNSBUS"
-		(at 102.87 87.63 0)
+	(label "BON"
+		(at 311.15 74.93 0)
 		(fields_autoplaced yes)
 		(effects
@@
 		)
 	)
-	(label "BT1"
+	(label "BTN1"
 		(at 330.2 80.01 0)
 		(fields_autoplaced yes)
@@
 		)
 	)
-	(label "OSCIN"
+	(label "XTALH"
 		(at 347.98 162.56 0)
 		(fields_autoplaced yes)
@@
 		)
 	)
-	(label "TSW1B"
-		(at 191.77 43.18 0)
+	(label "SNMOSI"
+		(at 367.03 74.93 0)
 		(fields_autoplaced yes)
 		(effects
@@
 		)
 	)
-	(label "SNMOSI"
-		(at 367.03 74.93 0)
+	(label "BON"
+		(at 100.33 111.76 0)
 		(fields_autoplaced yes)
 		(effects
@@
 		)
 	)
-	(label "OSCLO"
+	(label "XTALC"
 		(at 316.23 201.93 0)
 		(fields_autoplaced yes)
@@
 		)
 	)
-	(label "PWRON"
-		(at 100.33 111.76 0)
-		(fields_autoplaced yes)
-		(effects
-			(font
-				(size 1.27 1.27)
-			)
-			(justify left bottom)
-		)
-	)
-	(label "BT1"
+	(label "BTN1"
 		(at 175.26 58.42 0)
 		(fields_autoplaced yes)
@@
 		)
 	)
-	(label "BT2"
+	(label "BTN2"
 		(at 330.2 82.55 0)
 		(fields_autoplaced yes)
@@
 		)
 	)
-	(label "DRDY"
-		(at 340.36 74.93 0)
-		(fields_autoplaced yes)
-		(effects
-			(font
-				(size 1.27 1.27)
-			)
-			(justify left bottom)
-		)
-	)
-	(label "BT4"
+	(label "BTN4"
 		(at 200.66 77.47 0)
 		(fields_autoplaced yes)
@@
 		)
 	)
-	(label "OSCOUT"
+	(label "XTALL"
 		(at 332.74 201.93 0)
 		(fields_autoplaced yes)
@@
 		)
 	)
-	(label "TSW2B"
-		(at 217.17 43.18 0)
+	(label "SW1A"
+		(at 193.04 38.1 0)
 		(fields_autoplaced yes)
 		(effects
@@
 	)
 	(symbol
+		(lib_id "power:VDD")
+		(at 368.3 119.38 0)
+		(unit 1)
+		(exclude_from_sim no)
+		(in_bom yes)
+		(on_board yes)
+		(dnp no)
+		(fields_autoplaced yes)
+		(property "Reference" "#PWR04"
+			(at 368.3 123.19 0)
+			(effects
+				(font
+					(size 1.27 1.27)
+				)
+				(hide yes)
+			)
+		)
+		(property "Value" "+3V3"
+			(at 368.3 114.3 0)
+			(effects
+				(font
+					(size 1.27 1.27)
+				)
+			)
+		)
+		(property "Footprint" ""
+			(at 368.3 119.38 0)
+			(effects
+				(font
+					(size 1.27 1.27)
+				)
+				(hide yes)
+			)
+		)
+		(property "Datasheet" ""
+			(at 368.3 119.38 0)
+			(effects
+				(font
+					(size 1.27 1.27)
+				)
+				(hide yes)
+			)
+		)
+		(property "Description" "Power symbol creates a global label with name \"VDD\""
+			(at 368.3 119.38 0)
+			(effects
+				(font
+					(size 1.27 1.27)
+				)
+				(hide yes)
+			)
+		)
+		(pin "1"
+		)
+		(instances
+			(project "rc-controller"
+				(path "/194a9ee6-1a0c-43bb-8d51-0f60bff519bd"
+					(reference "#PWR04")
+					(unit 1)
+				)
+			)
+		)
+	)
+	(symbol
 		(lib_id "Device:C")
 		(at 77.47 257.81 0)
@@
 		(on_board yes)
 		(dnp no)
-		(fields_autoplaced yes)
 		(property "Reference" "C23"
 			(at 337.82 223.5199 0)
@@
 	)
 	(symbol
-		(lib_id "power:VDD")
-		(at 368.3 119.38 0)
-		(unit 1)
-		(exclude_from_sim no)
-		(in_bom yes)
-		(on_board yes)
-		(dnp no)
-		(fields_autoplaced yes)
-		(property "Reference" "#PWR04"
-			(at 368.3 123.19 0)
-			(effects
-				(font
-					(size 1.27 1.27)
-				)
-				(hide yes)
-			)
-		)
-		(property "Value" "+3V3"
-			(at 368.3 114.3 0)
-			(effects
-				(font
-					(size 1.27 1.27)
-				)
-			)
-		)
-		(property "Footprint" ""
-			(at 368.3 119.38 0)
-			(effects
-				(font
-					(size 1.27 1.27)
-				)
-				(hide yes)
-			)
-		)
-		(property "Datasheet" ""
-			(at 368.3 119.38 0)
-			(effects
-				(font
-					(size 1.27 1.27)
-				)
-				(hide yes)
-			)
-		)
-		(property "Description" "Power symbol creates a global label with name \"VDD\""
-			(at 368.3 119.38 0)
-			(effects
-				(font
-					(size 1.27 1.27)
-				)
-				(hide yes)
-			)
-		)
-		(pin "1"
-		)
-		(instances
-			(project "rc-controller"
-				(path "/194a9ee6-1a0c-43bb-8d51-0f60bff519bd"
-					(reference "#PWR04")
-					(unit 1)
-				)
-			)
-		)
-	)
-	(symbol
 		(lib_name "GND_2")
 		(lib_id "power:GND")
@@
 		(lib_name "GND_11")
 		(lib_id "power:GND")
-		(at 129.54 267.97 0)
+		(at 129.54 265.43 0)
 		(unit 1)
 		(exclude_from_sim no)
@@
 		(fields_autoplaced yes)
 		(property "Reference" "#PWR07"
-			(at 129.54 274.32 0)
+			(at 129.54 271.78 0)
 			(effects
 				(font
@@
 		)
 		(property "Value" "GND"
-			(at 129.54 273.05 0)
+			(at 129.54 270.51 0)
 			(effects
 				(font
@@
 		)
 		(property "Footprint" ""
-			(at 129.54 267.97 0)
+			(at 129.54 265.43 0)
 			(effects
 				(font
@@
 		)
 		(property "Datasheet" ""
-			(at 129.54 267.97 0)
+			(at 129.54 265.43 0)
 			(effects
 				(font
@@
 		)
 		(property "Description" "Power symbol creates a global label with name \"GND\" , ground"
-			(at 129.54 267.97 0)
+			(at 129.54 265.43 0)
 			(effects
 				(font

Commit message: Finish schematic
Parts:
- added H1, H2, H3, H4: MountingHole, MountingHole:MountingHole_3.2mm_M3, symbol Mechanical:MountingHole
- added J1: Conn_01x04_Pin, Connector_PinHeader_2.54mm:PinHeader_1x04_P2.54mm_Horizontal, symbol Connector:Conn_01x04_Pin
Connections:
- net RFMISO is gone; now on net SNMISO: U7.7 (MISO)
- net RFMOSI is gone; now on net SNMOSI: U7.6 (MOSI)
- net RFSCK is gone; now on net SNCLK: U7.5 (SCK)
- net SNSCK is gone; now on net SNCLK: U2.2 (SCL), U5.13 (SCL/SCLK)
- net +3V3: now also JY1.H1 (H+), JY1.V1 (V+), JY2.H1 (H+), JY2.V1 (V+), J1.4 (Pin_4); no longer JY1.A1 (XH), JY1.A2 (YH), JY2.A1 (XH), JY2.A2 (YH)
- net BON: now also U1.27 (PB1)
- net BREF: now also U1.24 (PC4)
- net BTN1: now also U1.56 (PB4)
- net BTN2: now also U1.57 (PB5)
- net BTN3: now also U1.26 (PB0)
- net BTN4: now also U1.17 (PA3)
- net CHRG: now also U1.38 (PC7)
- net GCS: now also U1.36 (PB15)
- net GND: now also JY1.H3 (H-), JY1.S1 (Shield), JY1.V3 (V-), JY2.H3 (H-), JY2.S1 (Shield), JY2.V3 (V-), J1.1 (Pin_1); no longer JY1.B1 (XL), JY1.MP (Shield), JY1.S2 (SWB), JY2.B1 (XL), JY2.MP (Shield), JY2.S2 (SWB)
- net JY1SW: now also JY1.B1 (SWA), U1.54 (PD2); no longer JY1.S1 (SWA)
- net JY1X: now also JY1.V2 (V), U1.9 (PC1); no longer JY1.C1 (X)
- net JY1Y: now also JY1.H2 (H), U1.8 (PC0); no longer JY1.C2 (Y)
- net JY2SW: now also JY2.B1 (SWA), U1.28 (PB2); no longer JY2.S1 (SWA)
- net JY2X: now also JY2.V2 (V), U1.10 (PC2); no longer JY2.C1 (X)
- net JY2Y: now also JY2.H2 (H), U1.11 (PC3); no longer JY2.C2 (Y)
- net MTR: now also U1.4 (PC15)
- net PCS: now also U1.62 (PB9)
- net RE1A: now also U1.52 (PC11)
- net RE1B: now also U1.53 (PC12)
- net RE1SW: now also U1.55 (PB3)
- net RE2A: now also U1.43 (PA10)
- net RE2B: now also U1.29 (PB10)
- net RE2SW: now also U1.3 (PC14)
- net RFCE: now also U1.33 (PB12)
- net RFCS: now also U1.35 (PB14)
- net SCL: now also U1.58 (PB6)
- net SDA: now also U1.59 (PB7)
- net SNMISO: now also U1.22 (PA6)
- net SNMOSI: now also U1.23 (PA7)
- net STDBY: now also U1.39 (PC8)
- net SW1A: now also U1.51 (PC10)
- net SW1B: now also U1.50 (PA15)
- net SW2A: now also U1.37 (PC6)
- net SW2B: now also U1.25 (PC5)
- net SNCLK: now reaches U1.21 (PA5)
- net SWDIO: now reaches U1.46 (PA13)
- net SWDIO: now also J1.3 (Pin_3)
- net SWCLK: now reaches U1.49 (PA14)
- net SWCLK: now also J1.2 (Pin_2)
- net DRDY: no longer names the net of U2.7 (INT_DRDY)
- net GINT1: no longer names the net of U5.4 (INT1)
- net RFIRQ: no longer names the net of U7.8 (IRQ)
- no-connect marks 6 -> 17
Other:
- note added: "Mounting"

Commit message: Fix bom and generate fab files
Parts:
- BT1, J1, JP1: now not fitted
- C14: footprint Capacitor_SMD:C_0402_1005Metric -> Capacitor_SMD:C_0603_1608Metric; LCSC (none) -> C1595
- D2, D4: LCSC (none) -> C7420362
- J2: LCSC (none) -> C165948
- R12: value 340k -> 330k; LCSC (none) -> C25778
- R9: value 1m -> 1M; LCSC (none) -> C26083
- U1: LCSC (none) -> C74524
- U4: LCSC (none) -> C448642
- U6: footprint Package_TO_SOT_SMD:TSOT-23-6 -> Package_TO_SOT_SMD:SOT-23-6
Connections:
- net GND: now also RE1.MP, RE2.MP
- no-connect marks 17 -> 18

Commit message: Initialize stm32 project and fix vref issue
Parts:
- U4: footprint Package_SO:SOP-8-1EP_4.57x4.57mm_P1.27mm_EP4.57x4.45mm -> Package_SO:HSOP-8-1EP_3.9x4.9mm_P1.27mm_EP2.41x3.1mm
Connections:
- net VREF is gone; now on net +3V3: C24.1, C25.1, U1.13 (VREF+)
Changed lines of the file:
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@@
 	)
 	(junction
+		(at 325.12 157.48)
+		(diameter 0)
+		(color 0 0 0 0)
+	)
+	(junction
 		(at 132.08 69.85)
 		(diameter 0)
@@
 	(wire
 		(pts
+			(xy 325.12 144.78) (xy 325.12 157.48)
+		)
+		(stroke
+			(width 0)
+			(type default)
+		)
+	)
+	(wire
+		(pts
 			(xy 36.83 104.14) (xy 41.91 104.14)
 		)
@@
 		)
 	)
-	(label "VREF"
-		(at 349.25 157.48 0)
-		(fields_autoplaced yes)
-		(effects
-			(font
-				(size 1.27 1.27)
-			)
-			(justify left bottom)
-		)
-	)
 	(label "USB_D+"
 		(at 83.82 190.5 0)
@@
 	)
 	(symbol
+		(lib_id "power:VDD")
+		(at 325.12 144.78 0)
+		(unit 1)
+		(exclude_from_sim no)
+		(in_bom yes)
+		(on_board yes)
+		(dnp no)
+		(fields_autoplaced yes)
+		(property "Reference" "#PWR086"
+			(at 325.12 148.59 0)
+			(effects
+				(font
+					(size 1.27 1.27)
+				)
+				(hide yes)
+			)
+		)
+		(property "Value" "+3V3"
+			(at 325.12 139.7 0)
+			(effects
+				(font
+					(size 1.27 1.27)
+				)
+			)
+		)
+		(property "Footprint" ""
+			(at 325.12 144.78 0)
+			(effects
+				(font
+					(size 1.27 1.27)
+				)
+				(hide yes)
+			)
+		)
+		(property "Datasheet" ""
+			(at 325.12 144.78 0)
+			(effects
+				(font
+					(size 1.27 1.27)
+				)
+				(hide yes)
+			)
+		)
+		(property "Description" "Power symbol creates a global label with name \"VDD\""
+			(at 325.12 144.78 0)
+			(effects
+				(font
+					(size 1.27 1.27)
+				)
+				(hide yes)
+			)
+		)
+		(pin "1"
+		)
+		(instances
+			(project "rc-controller"
+				(path "/194a9ee6-1a0c-43bb-8d51-0f60bff519bd"
+					(reference "#PWR086")
+					(unit 1)
+				)
+			)
+		)
+	)
+	(symbol
 		(lib_id "Device:R")
 		(at 146.05 107.95 0)
@@
 			)
 		)
-		(property "Footprint" "Package_SO:SOP-8-1EP_4.57x4.57mm_P1.27mm_EP4.57x4.45mm"
+		(property "Footprint" "Package_SO:HSOP-8-1EP_3.9x4.9mm_P1.27mm_EP2.41x3.1mm"
 			(at 63.754 76.962 0)
 			(effects

Commit message: Update charging circuitry
Parts:
- removed D4: SS24, Diode_SMD:D_SMA, symbol Diode:SS24
- removed J1: Conn_01x04_Pin, Connector_PinHeader_2.54mm:PinHeader_1x04_P2.54mm_Horizontal, symbol Connector:Conn_01x04_Pin
- removed JP1: Jumper_2_Open, Jumper:SolderJumper-2_P1.3mm_Open_RoundedPad1.0x1.5mm, symbol Jumper:Jumper_2_Open
- removed L1: 10u, Inductor_SMD:L_1206_3216Metric, symbol Device:L
- removed Q2: AO3401A, Package_TO_SOT_SMD:SOT-23, symbol Transistor_FET:AO3401A
- removed Q3, Q4: AO3400A, Package_TO_SOT_SMD:SOT-23, symbol Transistor_FET:AO3400A
- removed U2: LPS22HB, Package_LGA:ST_HLGA-10_2x2mm_P0.5mm_LayoutBorder3x2y, symbol Sensor_Pressure:LPS22HB
- removed U4: TX4401, Package_SO:HSOP-8-1EP_3.9x4.9mm_P1.27mm_EP2.41x3.1mm, symbol User_Symbols:TX4401
- removed U6: TP4057-42, Package_TO_SOT_SMD:SOT-23-6, symbol User_Symbols:TP4057-42
- added BT2: Battery_Cell, symbol Device:Battery_Cell
- added C29: 100u, symbol Device:C
- added D3: LEDG, symbol Device:LED
- added D4: SS34, Diode_SMD:D_SMA, symbol Diode:SS34
- added D5: LEDB, symbol Device:LED
- added J1: Conn_ARM_SWD_TagConnect_TC2030-NL, Connector:Tag-Connect_TC2030-IDC-NL_2x03_P1.27mm_Vertical, symbol Connector:Conn_ARM_SWD_TagConnect_TC2030-NL
- added Q10, Q11, Q6, Q7: AO3400A, Package_TO_SOT_SMD:SOT-23, symbol Transistor_FET:AO3400A
- added Q12, Q2: MDD2302, Package_TO_SOT_SMD:SOT-23, symbol User_Symbols:MDD2302
- added Q4, Q5, Q8, Q9: AO3401A, Package_TO_SOT_SMD:SOT-23, symbol Transistor_FET:AO3401A
- added R19, R20: 500, symbol Device:R
- added R21, R22: 4.7k, Resistor_SMD:R_0402_1005Metric, symbol Device:R
- added R23: 10k, symbol Device:R
- added U2: AT24CS32-SSHM, Package_SO:SOIC-8_3.9x4.9mm_P1.27mm, symbol Memory_EEPROM:AT24CS32-SSHM
- added U4: AMS1117-3.3, Package_TO_SOT_SMD:SOT-223-3_TabPin2, symbol Regulator_Linear:AMS1117-3.3
- added U6: ACS712xLCTR-05B, Package_SO:SOIC-8_3.9x4.9mm_P1.27mm, symbol Sensor_Current:ACS712xLCTR-05B
- BT1: footprint Connector_PinHeader_2.54mm:PinHeader_1x02_P2.54mm_Vertical -> (none); now fitted
- C12: value 10u -> 22u; footprint Capacitor_SMD:C_0603_1608Metric -> (none); LCSC C19702 -> (none)
- C13: value 100n -> 22u; footprint Capacitor_SMD:C_0402_1005Metric -> (none)
- C14: value 1n5 -> 100u; footprint Capacitor_SMD:C_0603_1608Metric -> Capacitor_SMD:C_1206_3216Metric; LCSC C1595 -> (none)
- C15: value 22u -> 1n; footprint Capacitor_SMD:C_0603_1608Metric -> (none)
- C16: value 10u -> 100n; footprint Capacitor_SMD:C_0603_1608Metric -> (none)
- C17: value 1u -> 100u; footprint Capacitor_SMD:C_0402_1005Metric -> (none)
- D1: value LEDB -> LEDR
- PB1: footprint Button_Switch_THT:SW_PUSH_6mm_H13mm -> (none); LCSC C2834892 -> C499339
- R10: value 15k -> 10M; footprint Resistor_SMD:R_0402_1005Metric -> (none)
- R11: value 200k -> 50k; footprint Resistor_SMD:R_0402_1005Metric -> (none)
- R12: value 330k -> 50k; footprint Resistor_SMD:R_0402_1005Metric -> (none); LCSC C25778 -> (none)
- R13, R14: value 47k -> 10M; footprint Resistor_SMD:R_0402_1005Metric -> (none)
- R15: value 2k -> 10k
- R16: value 200k -> 10k
- R17: value 200k -> 10k; footprint Resistor_SMD:R_0402_1005Metric -> (none)
- R7: value 56k -> 10k; footprint Resistor_SMD:R_0402_1005Metric -> (none)
- R8: value 4k7 -> 10M; footprint Resistor_SMD:R_0402_1005Metric -> (none)
- R9: value 1M -> 100k; footprint Resistor_SMD:R_0402_1005Metric -> (none); LCSC C26083 -> (none)
- SW3, SW4, SW5, SW6: LCSC C2834892 -> C2834912
Connections:
- net VBUS is gone; now on net VUSB: C9.1, J2.A4 (VBUS), J2.A9 (VBUS), J2.B4 (VBUS), J2.B9 (VBUS), R2.1, R3.1, U3.5 (VP)
- net +3V3: now also C14.1, D4.1 (K), J1.1 (VCC), Q9.3 (D), R21.1, R22.1, U2.8 (VCC); no longer C15.1, R12.1
- net BREF: now also BT1.1 (+), C17.1, R12.1, R14.2, BT2.2 (-), C29.2, Q12.3 (D), Q2.2 (S); no longer R16.1, R17.2, U1.24 (PC4)
- net BTN1: no longer U1.56 (PB4)
- net BTN2: no longer U1.57 (PB5)
- net BTN3: no longer U1.26 (PB0)
- net BTN4: no longer U1.17 (PA3)
- net GCS: no longer U1.36 (PB15)
- net GND: now also C14.2, M1.SH, R13.2, R9.2, D3.1 (K), D5.1 (K), J1.5 (GND), Q10.2 (S), Q11.2 (S), Q12.2 (S), Q6.2 (S), Q7.2 (S), R23.2, U2.1 (A0), U2.2 (A1), U2.3 (A2), U2.4 (GND), U2.7 (WP), U4.1 (GND), U6.5 (GND); no longer R11.2, R14.2, R16.2, R7.2, U8.4 (GND)
- net JY1SW: no longer U1.54 (PD2)
- net JY1X: no longer U1.9 (PC1)
- net JY1Y: no longer U1.8 (PC0)
- net JY2SW: no longer U1.28 (PB2)
- net JY2X: no longer U1.10 (PC2)
- net JY2Y: no longer U1.11 (PC3)
- net MTR: no longer U1.4 (PC15)
- net RE1A: no longer U1.52 (PC11)
- net RE1B: no longer U1.53 (PC12)
- net RE1SW: no longer U1.55 (PB3)
- net RE2A: no longer U1.43 (PA10)
- net RE2B: no longer U1.29 (PB10)
- net RE2SW: no longer U1.3 (PC14)
- net RFCE: no longer U1.33 (PB12)
- net RFCS: no longer U1.35 (PB14)
- net SCL: now also R22.2, U2.6 (SCL); no longer U1.58 (PB6), U8.2 (SCL)
- net SDA: now also R21.2, U2.5 (SDA); no longer U1.59 (PB7), U8.1 (SDA)
- net SNSBUS: now also R8.1, U1.43 (PA10), Q7.1 (G), Q8.1 (G)
- net SW1A: no longer U1.51 (PC10)
- net SW1B: no longer U1.50 (PA15)
- net SW2A: no longer U1.37 (PC6)
- net SW2B: no longer U1.25 (PC5)
- net SWCLK: now also J1.4 (SWCLK)
- net SWDIO: now also J1.2 (SWDIO)
- net VBATT: now also R11.2, BT2.1 (+), C29.1, Q2.3 (D), Q8.3 (D), U6.3 (IP-), U6.4 (IP-); no longer BT1.1 (+), C16.1, R13.1
- net at PB1.2: now also R10.2, Q10.3 (D), Q9.1 (G); no longer R13.2
- net at R10.1: now also R8.2, Q8.2 (S), Q9.2 (S); no longer C14.1
- net VUSB: now reaches C13.1
- net VUSB: now also C16.1, R17.1, Q4.2 (S), U4.3 (VI), U6.8 (VCC); no longer R9.2
- net CSNS: now reaches R15.1
- net CSNS: now also R16.2
- net GIRQ: now reaches U5.4 (INT1)
- net RFIRQ: now reaches U7.8 (IRQ)
- net at R7.1: now also C12.1, R9.1, Q5.2 (S), U4.2 (VO); no longer R8.2
- net BON: no longer names the net of U1.27 (PB1)
- net BON: no longer R14.1
- net CHRG: no longer names the net of U1.38 (PC7)
- net PCS: no longer names the net of U1.62 (PB9)
- net SNCLK renamed CLK
- net CLK: no longer U1.21 (PA5)
- net SNMISO renamed MISO
- net MISO: no longer U1.22 (PA6)
- net SNMOSI renamed MOSI
- net MOSI: no longer U1.23 (PA7)
- net STDBY: no longer names the net of U1.39 (PC8)
- removed net VPWR: C12.1, R17.1, R9.1
- net XTALC renamed XTALR
- net XTALH renamed XTALO
- net XTALO: now also U1.6 (PH1); no longer U1.5 (PH0)
- net XTALL renamed XTALI
- net XTALI: now also U1.5 (PH0); no longer U1.6 (PH1)
- net nRST renamed RST
- net RST: now also J1.3 (~{RESET})
- new net: Q11.3 (D), Q4.1 (G), R17.2
- new net: Q5.1 (G), Q7.3 (D), R7.2
- new net: D4.2 (A), Q5.3 (D)
- new net: R16.1, U6.7 (VIOUT)
- new net: Q4.3 (D), U6.1 (IP+), U6.2 (IP+)
- new net: C15.1, U6.6 (FILTER)
- new net: Q6.3 (D), U8.4 (GND)
- new net: D3.2 (A), R19.2
- new net: D5.2 (A), R20.2
- new net CRSW: Q11.1 (G), R23.1
- new net DPY: Q6.1 (G)
- new net DSC1: Q12.1 (G), R13.1
- new net DSC2: Q2.1 (G), R14.1
- new net IGN: Q10.1 (G)
- new net LEDCRG: R20.1
- new net LEDFULL: R19.1
- new net SCL2: U8.2 (SCL)
- new net SDA2: U8.1 (SDA)
- new net SWO: J1.6 (SWO)
- now unconnected: R11.1, R12.2
- no-connect marks 18 -> 5
Other:
- note added: "EEPROM"
- note added: "FIX JOYSTICKS"
- note added: "Low Vgs(th), 0.6V typ, 1V max"
- note added: "Max 1nF capacitance"
- note removed: "Pressure Sensor"
- moved on the sheet: C1, C10, C11, C18, C19, C20, C21, C9, D1, H1, H2, H3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
