File: pcb/rc-controller.kicad_sch (KiCad schematic)
At the start: 98 parts, among them J1 Conn_ARM_SWD_TagConnect_TC203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, J2 USB_C_Receptacle_USB2.0_16P, M1 Motor_DC, Q1 AO3401A, Q10 AO3400A, Q11 AO3400A, Q12 MDD2302, Q2 MDD2302, Q4 AO3401A, Q5 AO3401A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

Commit message: Save
Parts:
- removed BT1, BT2: Battery_Cell, symbol Device:Battery_Cell
- removed Q11: AO3400A, Package_TO_SOT_SMD:SOT-23, symbol Transistor_FET:AO3400A
- removed Q4: AO3401A, Package_TO_SOT_SMD:SOT-23, symbol Transistor_FET:AO3401A
- added BT1, BT2: BH-AA-A5BJ012, User_Footprints:BH-AA-A5BJ012, symbol User_Symbols:BH-AA-A5BJ012
- added C30: C, symbol Device:C
- added C31: 100n, symbol Device:C
- added Q11: SS8050, symbol Simulation_SPICE:NPN
- added Q4: MJD127T4, symbol Simulation_SPICE:PNP
- added R24, R25: 10, symbol Device:R
- added U10: NE5532, symbol Amplifier_Operational:NE5532
- L2: value 2.2u -> 2u2
- R15: value 10k -> 4k7
- R16: value 10k -> 3k3
- R17: value 10k -> 10
- R23: value 10k -> 400
Connections:
- net BREF: now also BT1.1 (+), BT2.2 (-), R24.2; no longer Q12.3 (D)
- net CRSW: no longer R23.1
- net GND: now also BT1.2 (-), C30.2, C31.2, Q11.3 (E), U10.4 (V-); no longer R23.2
- net VBATT: now also BT2.1 (+), R25.2; no longer Q2.3 (D)
- net VUSB: now also C31.1, Q4.3 (E), U10.8 (V+); no longer R17.1
- net at R17.2: now also C30.1, U10.3 (+)
- net at U6.1 (IP+), U6.2 (IP+): now also Q4.1 (C)
- new net: Q11.1 (C), Q4.2 (B)
- new net: Q11.2 (B), R23.2
- new net: Q2.3 (D), R25.1
- new net: Q12.3 (D), R24.1
- new net: R23.1, U10.1, U10.2 (-)
- new net CTRL: R17.1
- no-connect marks 5 -> 8
Other:
- note added: "<-"
- moved on the sheet: C1, C10, C11, C12, C13, C14, C15, C16, C17, C18, C19, C2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
